File: hardware/FrontPanelMonoPCB.brd (EAGLE design)
At the start: 70.8 x 128.5 mm, 0 parts

Commit message: Frontpanel basic finished
Parts:
- added E$1: (no value), oshw:OSHW_8MM
Routing:
- net S$20: track 101.3 -> 0.00 mm
- net S$16: track 28.4 -> 0.00 mm
- net S$17: track 28.4 -> 0.00 mm
- net S$4: track 19.7 -> 48.0 mm
- net S$18: track 21.1 -> 0.00 mm
- net S$19: track 21.1 -> 0.00 mm
- net S$5: track 19.7 -> 0.00 mm
- net S$11: track 19.7 -> 0.00 mm
- net S$7: track 19.7 -> 0.00 mm
- net S$6: track 19.7 -> 0.00 mm
- net S$13: track 19.7 -> 0.00 mm
- net S$12: track 19.7 -> 0.00 mm
- net S$10: track 19.7 -> 0.00 mm
- net S$8: track 19.7 -> 0.00 mm
- net S$14: track 19.7 -> 0.00 mm
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- added copper zone on layer 1, net GDN
- added copper zone on layer 16, net GDN
- added copper zone on layer 16, net S$1
Other:
- board text added: "MONOMANIC EDITION"
- board text added: "a"
- board text added: "a collaborative open-source project by Patrick Dowling, mxmxmx, and Tim Churches."
- board text added: "b"
- board text added: "c"
- board text added: "cv"
- board text added: "d"
- board text added: "ornament & crime (o_C)"
- board text added: "trig"
